File: TP_Integrador/Archivos/KiCad/Amplificador.kicad_pcb (KiCad board)
At the start: 2 copper layers, 100 x 50 mm, 33 parts, among them J1 Conn_01x02_Pin, J2 Conn_01x01_Pin, J3 Conn_01x01_Pin, J4 Conn_01x01_Pin, J5 Conn_01x01_Pin, J6 Conn_01x01_Pin, Q1 BC547, Q10 TIP122, Q11 TIP127, Q2 BC547, Q3 BC557, Q4 BC557, Q5 BC547, Q6 BC547, Q7 BD140, Q8 BC547, Q9 BC547

Commit message: TP Integrador
Parts:
- added J10: Pin_Vo, Connector_PinHeader_2.54mm:PinHeader_1x01_P2.54mm_Vertical, F.Cu at (148.5, 84.0)
- added J11: Pin_GND, Connector_PinHeader_2.54mm:PinHeader_1x01_P2.54mm_Vertical, F.Cu at (122.5, 118.0)
- added J12: Jumper Realimentacion, Connector_PinHeader_2.54mm:PinHeader_1x02_P2.54mm_Vertical, F.Cu at (141.7, 89.0)
- added J7: Jumper Salida Etapa 1, Connector_PinHeader_2.54mm:PinHeader_1x02_P2.54mm_Vertical, F.Cu at (137.0, 101.7)
- added J8: Jumper Salida Pos Etapa 2, Connector_PinHeader_2.54mm:PinHeader_1x02_P2.54mm_Vertical, F.Cu at (157.0, 102.5)
- added J9: Jumper Salida Neg Etapa 2, Connector_PinHeader_2.54mm:PinHeader_1x02_P2.54mm_Vertical, F.Cu at (145.5, 115.7)
- J1: value Conn_01x02_Pin -> Bornera_Salida
- J2: value Conn_01x01_Pin -> Pin_Entrada
- J3: value Conn_01x01_Pin -> Pin_Vee
- J4: value Conn_01x01_Pin -> Pin_Vcc
- J5, J6: value Conn_01x01_Pin -> Pin_GND
- Q9: value BC547 -> BD139; footprint Package_TO_SOT_THT:TO-92_Inline -> Package_TO_SOT_THT:TO-126-3_Vertical
- moved J6 44.4 mm to (138.5, 84.0)
- moved R9 22.4 mm to (153.5, 95.9), turned to -90 degrees
- moved Q11 19.0 mm to (151.0, 116.0)
- moved Q10 15.6 mm to (163.0, 114.5)
- moved Q9 13.5 mm to (155.8, 109.6), turned to 180 degrees
- moved R8 12.1 mm to (149.0, 106.1), turned to 90 degrees
- moved R10 10.4 mm to (137.5, 124.7), turned to 180 degrees
- moved J2 9.50 mm to (125.5, 107.0)
- moved Q8 9.05 mm to (132.5, 110.5)
- moved J1 7.00 mm to (162.5, 87.0)
- moved Q7 6.10 mm to (141.0, 101.4)
- moved C3 5.12 mm to (145.0, 106.0)
- moved R7 4.50 mm to (118.0, 104.9)
- moved C2 4.24 mm to (130.5, 104.9), turned to 0 degrees
- moved R11 3.00 mm to (123.9, 94.0)
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Connections:
- C3 pad 1: /Vo1 -> /Entrada_Etapa_2
- C3 pad 2: /+Vo2 -> /Salida_Pos_Etapa_2
- Q10 pad 1: /+Vo2 -> /Entrada_Pos_Etapa_3
- Q11 pad 1: /-Vo2 -> /Entrada_Neg_Etapa_3
- Q2 pad 1: /Vo1 -> /Salida_Etapa_1
- Q4 pad 3: /Vo1 -> /Salida_Etapa_1
- Q7 pad 2: /+Vo2 -> /Salida_Pos_Etapa_2
- Q7 pad 3: /Vo1 -> /Entrada_Etapa_2
- Q8 pad 1: /-Vo2 -> /Salida_Neg_Etapa_2
- Q9 pad 1: /+Vo2 -> /Salida_Neg_Etapa_2
- Q9 pad 2: Net-(Q9-B) -> /Salida_Pos_Etapa_2
- Q9 pad 3: /-Vo2 -> Net-(Q9-B)
- R6 pad 1: /Vo -> Net-(J12-Pin_1)
- R8 pad 1: /+Vo2 -> /Salida_Pos_Etapa_2
- R9 pad 2: /-Vo2 -> /Salida_Neg_Etapa_2
Routing:
- net /Salida_Pos_Etapa_2: track 0.00 -> 51.1 mm
- net /-Vo2: track 45.4 -> 0.00 mm
- net /+Vo2: track 44.6 -> 0.00 mm
- net /Salida_Neg_Etapa_2: track 0.00 -> 38.3 mm
- net /Vo1: track 34.2 -> 0.00 mm
- net /Vcc: track 90.7 -> 115.7 mm
- net /Salida_Etapa_1: track 0.00 -> 23.5 mm
- net Net-(Q10-E): track 34.1 -> 12.4 mm
- net Net-(Q11-E): track 15.7 -> 32.6 mm
- net Net-(J12-Pin_1): track 0.00 -> 16.4 mm
- net /Vo: track 59.5 -> 44.1 mm
- net /Entrada_Pos_Etapa_3: track 0.00 -> 13.7 mm
- net /Vee: track 92.8 -> 80.1 mm
- net /VB_Q6: track 58.2 -> 46.6 mm
- net /Entrada_Etapa_2: track 0.00 -> 9.44 mm
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Other:
- board text added: "Alterino, Thiago Aksman, Ezequiel Beltrame, Alejo"
