File: TP_Integrador/Archivos/KiCad/Amplificador.kicad_sch (KiCad schematic)
At the start: 33 parts, among them J1 Conn_01x02_Pin, J2 Conn_01x01_Pin, J3 Conn_01x01_Pin, J4 Conn_01x01_Pin, J5 Conn_01x01_Pin, J6 Conn_01x01_Pin, Q1 BC547, Q10 TIP122, Q11 TIP127, Q2 BC547, Q3 BC557, Q4 BC557, Q5 BC547, Q6 BC547, Q7 BD140, Q8 BC547, Q9 BC547

Commit message: TP Integrador
Parts:
- removed Q9: BC547, Package_TO_SOT_THT:TO-92_Inline, symbol Transistor_BJT:BC547
- added J10: Pin_Vo, Connector_PinHeader_2.54mm:PinHeader_1x01_P2.54mm_Vertical, symbol Connector:Conn_01x01_Pin
- added J11: Pin_GND, Connector_PinHeader_2.54mm:PinHeader_1x01_P2.54mm_Vertical, symbol Connector:Conn_01x01_Pin
- added J12: Jumper Realimentacion, Connector_PinHeader_2.54mm:PinHeader_1x02_P2.54mm_Vertical, symbol Connector:Conn_01x02_Pin
- added J7: Jumper Salida Etapa 1, Connector_PinHeader_2.54mm:PinHeader_1x02_P2.54mm_Vertical, symbol Connector:Conn_01x02_Pin
- added J8: Jumper Salida Pos Etapa 2, Connector_PinHeader_2.54mm:PinHeader_1x02_P2.54mm_Vertical, symbol Connector:Conn_01x02_Pin
- added J9: Jumper Salida Neg Etapa 2, Connector_PinHeader_2.54mm:PinHeader_1x02_P2.54mm_Vertical, symbol Connector:Conn_01x02_Pin
- added Q9: BD139, Package_TO_SOT_THT:TO-126-3_Vertical, symbol Transistor_BJT:BD139
- J1: value Conn_01x02_Pin -> Bornera_Salida
- J2: value Conn_01x01_Pin -> Pin_Entrada
- J3: value Conn_01x01_Pin -> Pin_Vee
- J4: value Conn_01x01_Pin -> Pin_Vcc
- J5, J6: value Conn_01x01_Pin -> Pin_GND
Connections:
- net GND: now also J11.1 (Pin_1)
- net Vo: now also J10.1 (Pin_1), J12.2 (Pin_2); no longer R6.1
- net at R8.2, R9.1: now also Q9.3 (B)
- net +Vo2 renamed Salida_Pos_Etapa_2
- net Salida_Pos_Etapa_2: now also J8.1 (Pin_1), Q9.2 (C); no longer Q10.1 (B)
- net -Vo2 renamed Salida_Neg_Etapa_2
- net Salida_Neg_Etapa_2: now also J9.1 (Pin_1), Q9.1 (E); no longer Q11.1 (B)
- net Vo1 renamed Entrada_Etapa_2
- net Entrada_Etapa_2: now also J7.2 (Pin_2); no longer Q2.1 (C), Q4.3 (E)
- new net: J12.1 (Pin_1), R6.1
- new net Entrada_Neg_Etapa_3: J9.2 (Pin_2), Q11.1 (B)
- new net Entrada_Pos_Etapa_3: J8.2 (Pin_2), Q10.1 (B)
- new net Salida_Etapa_1: J7.1 (Pin_1), Q2.1 (C), Q4.3 (E)
Other:
- moved on the sheet: J6
